File: project_02/ENGI301_synthesizer.brd (EAGLE design)
At the start: 152.4 x 76.2 mm, 37 parts, among them SW1 SLIDE_SWITCH, SW2 SLIDE_SWITCH, U1 POCKETBEAGLE

Commit message: Made Board
Parts:
- removed U$1, U$2, U$3, U$4, U$7: ROT_POTENTIOMETER, ENGI301:POT-P102
- removed U$10, U$5, U$9: SPEAKER_30MM, ENGI301:SPEAKER_30MM
- added POT1, POT2, POT3, POT4, POT5: ROT_POTENTIOMETER, ENGI301:POT-P102
- added R10, R11, R12, R8, R9: (no value), ENGI301:R1210
- added SP1, SP2, SP3: SPEAKER_30MM, ENGI301:SPEAKER_30MM
- moved SW1 314.0 mm to (188.0, 66.0), turned to 180 degrees
- moved SW2 277.2 mm to (66.0, 66.0)
- moved R7 275.3 mm to (185.4, 12.7), turned to 90 degrees
- moved B 266.4 mm to (177.8, 25.4)
- moved AS 259.3 mm to (165.1, 45.7)
- moved A 226.0 mm to (152.4, 25.4)
- moved R6 222.4 mm to (160.0, 12.7), turned to 90 degrees
- moved GS 202.9 mm to (139.7, 45.7)
- moved R5 197.9 mm to (134.6, 12.7), turned to 90 degrees
- moved G 192.7 mm to (127.0, 25.4)
- moved R4 181.7 mm to (109.2, 12.7), turned to 90 degrees
- moved FS 173.0 mm to (114.3, 45.7)
- moved F 162.5 mm to (101.6, 25.4)
- moved U1 151.9 mm to (2.54, 114.3), flipped to the bottom
- moved E 129.2 mm to (76.2, 25.4)
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Connections:
- removed net I2C_SCL: U1.28
- removed net I2C_SDA: U1.26
- new net N$11: FS.1, FS.3, R10.2
- new net N$13: DS.1, DS.3, R11.2
- new net N$14: CS.1, CS.3, R12.2
- new net N$5: AS.1, AS.3, R8.2
- new net N$9: GS.1, GS.3, R9.2
- net A: now also U1.56; no longer U1.44
- net AIN_VREFN: now also POT3.CCW, POT4.CCW; no longer U$3.CCW, U$4.CCW
- net AIN_VREFP: now also POT3.CW, POT4.CW; no longer U$3.CW, U$4.CW
- net AS: now also U1.60; no longer U1.56
- net B: now also U1.20; no longer U1.53
- net C: now also U1.38; no longer U1.20
- net CS: now also U1.40; no longer U1.55
- net D: now also U1.42; no longer U1.60
- net DS: now also U1.46; no longer U1.58
- net E: now also U1.44; no longer U1.54
- net F: now also U1.53; no longer U1.46
- net FS: now also U1.55; no longer U1.42
- net G: now also U1.54; no longer U1.40
- net GND: now also SP1.-, SP2.-, SP3.-; no longer U$10.-, U$5.-, U$9.-
- net GS: now also U1.58; no longer U1.38
- net MAIN_SPEAK: now also POT1.S; no longer U$1.S
- net N$1: no longer CS.1, CS.3
- net N$10: now also POT1.CW, SP3.+; no longer U$1.CW, U$5.+
- net N$12: no longer GS.1, GS.3
- net N$15: no longer AS.1, AS.3
- net N$2: no longer DS.1, DS.3
- net N$3: now also POT5.CW, SP1.+; no longer U$2.CW, U$9.+
- net N$4: now also POT5.S; no longer U$2.S
- net N$6: now also POT2.CW, SP2.+; no longer U$10.+, U$7.CW
- net N$8: no longer FS.1, FS.3
- net REC_SPEAK: now also POT2.S; no longer U$7.S
- net TEMPO_SIG: now also POT4.S; no longer U$4.S
- net TIMBRE_SIG: now also POT3.S; no longer U$3.S
- net VDD_3P3V: now also R10.1, R11.1, R12.1, R8.1, R9.1
Routing:
- net B: track 0.00 -> 245.2 mm
- net REC_SW: track 0.00 -> 159.2 mm
- net A: track 0.00 -> 155.4 mm
- net AS: track 0.00 -> 151.4 mm
- net AIN_VREFP: track 0.00 -> 143.1 mm
- net G: track 0.00 -> 133.7 mm
- net AIN_VREFN: track 0.00 -> 131.1 mm
- net GS: track 0.00 -> 128.5 mm
- net REC_SPEAK: track 0.00 -> 126.4 mm
- net F: track 0.00 -> 117.2 mm
- net FS: track 0.00 -> 113.5 mm
- net MAIN_SPEAK: track 0.00 -> 103.7 mm
- net TIMBRE_SIG: track 0.00 -> 100.1 mm
- net E: track 0.00 -> 99.2 mm
- net D: track 0.00 -> 89.4 mm
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Other:
- board size 152.4 x 76.2 mm -> 203.2 x 127 mm

Commit message: no message
Parts:
- R1, R10, R11, R12, R2, R3, R4, R5, R6, R7, R8, R9: value (none) -> 10k
- moved SW2 7.62 mm to (66.0, 73.7)
Connections:
- net VDD_5V renamed VOUT
Routing:
- net MAIN_SPEAK: track 103.7 -> 97.9 mm
- net N$4: track 34.0 -> 31.0 mm
- net GND: track 26.1 -> 28.4 mm
Other:
- board text added: "JS"
- board text added: "Main Volume"
- board text added: "Met Power"
- board text added: "Met Volume"
- board text added: "Pocket Synthesizer"
- board text added: "Record"
- board text added: "Recording Volume"
- board text added: "Rev. 1-A"
- board text added: "Tempo"
- board text added: "Timbre"
