File: project_02/ENGI301_synthesizer.sch (EAGLE design)
At the start: 37 parts, among them SW1 SLIDE_SWITCH, SW2 SLIDE_SWITCH, U1 POCKETBEAGLE

Commit message: Made Board
Parts:
- removed U$1, U$7: ROT_POTENTIOMETER, ENGI301:ROT_POTENTIOMETER
- removed U$10, U$5: SPEAKER_30MM, ENGI301:SPEAKER_30MM
- added POT1, POT2: ROT_POTENTIOMETER, ENGI301:ROT_POTENTIOMETER
- added R10, R11, R12, R8, R9: (no value), ENGI301:R_R1210
- added SP2, SP3: SPEAKER_30MM, ENGI301:SPEAKER_30MM
- renumbered U$2 to POT5, U$3 to POT3, U$4 to POT4, U$9 to SP1
Connections:
- removed net I2C_SCL: U1.I2C2.SCL
- removed net I2C_SDA: U1.I2C2.SDA
- new net N$11: FS.1, FS.3, R10.2
- new net N$13: DS.1, DS.3, R11.2
- new net N$14: CS.1, CS.3, R12.2
- new net N$5: AS.1, AS.3, R8.2
- new net N$9: GS.1, GS.3, R9.2
- net A: now also U1.GPIO64; no longer U1.GPIO60
- net AS: now also U1.GPIO44; no longer U1.GPIO64
- net B: now also U1.GPIO20; no longer U1.GPIO65
- net C: now also U1.GPIO59; no longer U1.GPIO20
- net CS: now also U1.GPIO58; no longer U1.GPIO27
- net D: now also U1.GPIO57; no longer U1.GPIO44
- net DS: now also U1.GPIO52; no longer U1.GPIO46
- net E: now also U1.GPIO60; no longer U1.GPIO47
- net F: now also U1.GPIO65; no longer U1.GPIO52
- net FS: now also U1.GPIO27; no longer U1.GPIO57
- net G: now also U1.GPIO47; no longer U1.GPIO58
- net GND: now also SP2.-, SP3.-; no longer U$10.-, U$5.-
- net GS: now also U1.GPIO46; no longer U1.GPIO59
- net MAIN_SPEAK: now also POT1.WIPER; no longer U$1.WIPER
- net N$1: no longer CS.1, CS.3
- net N$10: now also POT1.CW, SP3.+; no longer U$1.CW, U$5.+
- net N$12: no longer GS.1, GS.3
- net N$15: no longer AS.1, AS.3
- net N$2: no longer DS.1, DS.3
- net N$6: now also POT2.CW, SP2.+; no longer U$10.+, U$7.CW
- net N$8: no longer FS.1, FS.3
- net REC_SPEAK: now also POT2.WIPER; no longer U$7.WIPER
- net VDD_3P3V: now also R10.1, R11.1, R12.1, R8.1, R9.1
Other:
- moved on the sheet: A, AS, B, C, CS, D, DS, E, F, FS, G, GS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

Commit message: no message
Parts:
- R1, R10, R11, R12, R2, R3, R4, R5, R6, R7, R8, R9: value (none) -> 10k
Connections:
- removed net VDD_5V: U1.VOUT@1, U1.VOUT@2
Other:
- note added: "1 of 1"
- note added: "Josh Stelling"
- note added: "Pocket Synthesizer"
Changed lines of the file:
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@@
 <part name="SUPPLY1" library="ENGI301" deviceset="VDD_3P3V" device=""/>
 <part name="SUPPLY4" library="ENGI301" deviceset="VDD_3P3V" device=""/>
-<part name="SUPPLY3" library="ENGI301" deviceset="VDD_5V" device=""/>
-<part name="SUPPLY2" library="ENGI301" deviceset="VDD_5V" device=""/>
 <part name="MGT1" library="ENGI301" deviceset="MOUNTING_HOLE" device=""/>
 <part name="MGT2" library="ENGI301" deviceset="MOUNTING_HOLE" device=""/>
@@
 <part name="C" library="ENGI301" deviceset="PUSH_BUTTON" device=""/>
 <part name="CS" library="ENGI301" deviceset="PUSH_BUTTON" device=""/>
-<part name="R1" library="ENGI301" deviceset="R_" device="R1210"/>
+<part name="R1" library="ENGI301" deviceset="R_" device="R1210" value="10k"/>
 <part name="SUPPLY5" library="ENGI301" deviceset="VDD_3P3V" device=""/>
 <part name="D" library="ENGI301" deviceset="PUSH_BUTTON" device=""/>
 <part name="DS" library="ENGI301" deviceset="PUSH_BUTTON" device=""/>
-<part name="R2" library="ENGI301" deviceset="R_" device="R1210"/>
+<part name="R2" library="ENGI301" deviceset="R_" device="R1210" value="10k"/>
 <part name="SUPPLY6" library="ENGI301" deviceset="VDD_3P3V" device=""/>
 <part name="E" library="ENGI301" deviceset="PUSH_BUTTON" device=""/>
-<part name="R3" library="ENGI301" deviceset="R_" device="R1210"/>
+<part name="R3" library="ENGI301" deviceset="R_" device="R1210" value="10k"/>
 <part name="SUPPLY7" library="ENGI301" deviceset="VDD_3P3V" device=""/>
 <part name="F" library="ENGI301" deviceset="PUSH_BUTTON" device=""/>
 <part name="FS" library="ENGI301" deviceset="PUSH_BUTTON" device=""/>
-<part name="R4" library="ENGI301" deviceset="R_" device="R1210"/>
+<part name="R4" library="ENGI301" deviceset="R_" device="R1210" value="10k"/>
 <part name="SUPPLY8" library="ENGI301" deviceset="VDD_3P3V" device=""/>
 <part name="G" library="ENGI301" deviceset="PUSH_BUTTON" device=""/>
 <part name="GS" library="ENGI301" deviceset="PUSH_BUTTON" device=""/>
-<part name="R5" library="ENGI301" deviceset="R_" device="R1210"/>
+<part name="R5" library="ENGI301" deviceset="R_" device="R1210" value="10k"/>
 <part name="SUPPLY9" library="ENGI301" deviceset="VDD_3P3V" device=""/>
 <part name="A" library="ENGI301" deviceset="PUSH_BUTTON" device=""/>
 <part name="AS" library="ENGI301" deviceset="PUSH_BUTTON" device=""/>
-<part name="R6" library="ENGI301" deviceset="R_" device="R1210"/>
+<part name="R6" library="ENGI301" deviceset="R_" device="R1210" value="10k"/>
 <part name="SUPPLY10" library="ENGI301" deviceset="VDD_3P3V" device=""/>
 <part name="B" library="ENGI301" deviceset="PUSH_BUTTON" device=""/>
-<part name="R7" library="ENGI301" deviceset="R_" device="R1210"/>
+<part name="R7" library="ENGI301" deviceset="R_" device="R1210" value="10k"/>
 <part name="SUPPLY11" library="ENGI301" deviceset="VDD_3P3V" device=""/>
 <part name="SUPPLY12" library="ENGI301" deviceset="VDD_3P3V" device=""/>
@@
 <part name="GND5" library="ENGI301" deviceset="GND" device=""/>
 <part name="GND6" library="ENGI301" deviceset="GND" device=""/>
-<part name="R8" library="ENGI301" deviceset="R_" device="R1210"/>
+<part name="R8" library="ENGI301" deviceset="R_" device="R1210" value="10k"/>
 <part name="SUPPLY13" library="ENGI301" deviceset="VDD_3P3V" device=""/>
-<part name="R9" library="ENGI301" deviceset="R_" device="R1210"/>
+<part name="R9" library="ENGI301" deviceset="R_" device="R1210" value="10k"/>
 <part name="SUPPLY14" library="ENGI301" deviceset="VDD_3P3V" device=""/>
-<part name="R10" library="ENGI301" deviceset="R_" device="R1210"/>
+<part name="R10" library="ENGI301" deviceset="R_" device="R1210" value="10k"/>
 <part name="SUPPLY15" library="ENGI301" deviceset="VDD_3P3V" device=""/>
-<part name="R11" library="ENGI301" deviceset="R_" device="R1210"/>
+<part name="R11" library="ENGI301" deviceset="R_" device="R1210" value="10k"/>
 <part name="SUPPLY16" library="ENGI301" deviceset="VDD_3P3V" device=""/>
-<part name="R12" library="ENGI301" deviceset="R_" device="R1210"/>
+<part name="R12" library="ENGI301" deviceset="R_" device="R1210" value="10k"/>
 <part name="SUPPLY17" library="ENGI301" deviceset="VDD_3P3V" device=""/>
 <part name="POT1" library="ENGI301" deviceset="ROT_POTENTIOMETER" device=""/>
@@
 <wire x1="289.56" y1="114.3" x2="289.56" y2="187.96" width="0.3048" layer="97"/>
 <wire x1="142.24" y1="35.56" x2="378.46" y2="35.56" width="0.3048" layer="97"/>
+<text x="246.38" y="12.7" size="5.08" layer="97">Pocket Synthesizer</text>
+<text x="325.628" y="5.334" size="2.54" layer="97">1 of 1</text>
+<text x="313.182" y="20.32" size="2.54" layer="97">Josh Stelling</text>
 </plain>
 <instances>
@@
 <attribute name="VALUE" x="111.76" y="174.244" size="1.778" layer="96" align="center"/>
 </instance>
-<instance part="SUPPLY3" gate="G$1" x="99.06" y="170.18" smashed="yes">
-<attribute name="VALUE" x="99.06" y="174.244" size="1.778" layer="96" align="center"/>
-</instance>
-<instance part="SUPPLY2" gate="G$1" x="33.02" y="170.18" smashed="yes">
-<attribute name="VALUE" x="33.02" y="174.244" size="1.778" layer="96" align="center"/>
-</instance>
 <instance part="MGT1" gate="G$1" x="119.38" y="20.32" smashed="yes">
 <attribute name="NAME" x="120.142" y="18.288" size="1.27" layer="95"/>
@@
 <instance part="R2" gate="G$1" x="81.28" y="231.14" smashed="yes" rot="R270">
 <attribute name="NAME" x="78.74" y="233.68" size="1.778" layer="95" rot="R270"/>
-<attribute name="VALUE" x="76.2" y="233.68" size="1.778" layer="96" rot="R270"/>
+<attribute name="VALUE" x="78.74" y="228.6" size="1.778" layer="96" rot="R270"/>
 </instance>
 <instance part="SUPPLY6" gate="G$1" x="81.28" y="241.3" smashed="yes">
@@
 <instance part="R3" gate="G$1" x="137.16" y="231.14" smashed="yes" rot="R270">
 <attribute name="NAME" x="134.62" y="233.68" size="1.778" layer="95" rot="R270"/>
-<attribute name="VALUE" x="132.08" y="233.68" size="1.778" layer="96" rot="R270"/>
+<attribute name="VALUE" x="134.62" y="228.6" size="1.778" layer="96" rot="R270"/>
 </instance>
 <instance part="SUPPLY7" gate="G$1" x="137.16" y="241.3" smashed="yes">
@@
 <instance part="R5" gate="G$1" x="231.14" y="231.14" smashed="yes" rot="R270">
 <attribute name="NAME" x="228.6" y="233.68" size="1.778" layer="95" rot="R270"/>
-<attribute name="VALUE" x="226.06" y="233.68" size="1.778" layer="96" rot="R270"/>
+<attribute name="VALUE" x="228.6" y="228.6" size="1.778" layer="96" rot="R270"/>
 </instance>
 <instance part="SUPPLY9" gate="G$1" x="231.14" y="241.3" smashed="yes">
@@
 <instance part="R6" gate="G$1" x="287.02" y="231.14" smashed="yes" rot="R270">
 <attribute name="NAME" x="284.48" y="233.68" size="1.778" layer="95" rot="R270"/>
-<attribute name="VALUE" x="281.94" y="233.68" size="1.778" layer="96" rot="R270"/>
+<attribute name="VALUE" x="284.48" y="228.6" size="1.778" layer="96" rot="R270"/>
 </instance>
 <instance part="SUPPLY10" gate="G$1" x="287.02" y="241.3" smashed="yes">
@@
 <instance part="R7" gate="G$1" x="342.9" y="231.14" smashed="yes" rot="R270">
 <attribute name="NAME" x="340.36" y="233.68" size="1.778" layer="95" rot="R270"/>
-<attribute name="VALUE" x="337.82" y="233.68" size="1.778" layer="96" rot="R270"/>
+<attribute name="VALUE" x="340.36" y="228.6" size="1.778" layer="96" rot="R270"/>
 </instance>
 <instance part="SUPPLY11" gate="G$1" x="342.9" y="241.3" smashed="yes">
@@
 </segment>
 </net>
-<net name="VDD_5V" class="0">
-<segment>
-<pinref part="U1" gate="G$1" pin="VOUT@1"/>
-<pinref part="SUPPLY2" gate="G$1" pin="VDD_5V"/>
-<wire x1="40.64" y1="162.56" x2="33.02" y2="162.56" width="0.1524" layer="91"/>
-<wire x1="33.02" y1="162.56" x2="33.02" y2="167.64" width="0.1524" layer="91"/>
-</segment>
-<segment>
-<pinref part="U1" gate="G$1" pin="VOUT@2"/>
-<pinref part="SUPPLY3" gate="G$1" pin="VDD_5V"/>
-<wire x1="91.44" y1="162.56" x2="99.06" y2="162.56" width="0.1524" layer="91"/>
-<wire x1="99.06" y1="162.56" x2="99.06" y2="167.64" width="0.1524" layer="91"/>
-</segment>
-</net>
